Commit message: Version fonctionelle utilisant diff_drive_controller afin que le robot se stop lorsqu'aucune touche n'a été appuyée pendant un certain temps

File: dummiebot_description/urdf/macros.xacro (robot description, xacro)
@@ -57,4 +57,5 @@
       <joint_properties damping="0.0" friciton="0.0"/>
     </joint>
+<!--
     <transmission name="${lr}_trans">
       <type>transmission_interface/SimpleTransmission</type>
@@ -67,4 +68,15 @@
       </actuator>
     </transmission>
+-->
+    <transmission name="${lr}_trans">
+      <type>transmission_interface/SimpleTransmission</type>
+      <joint name="${lr}_wheel_hinge">
+        <hardwareInterface>hardware_interface/VelocityJointInterface</hardwareInterface>
+      </joint>
+      <actuator name="${lr}_motor">
+        <hardwareInterface>hardware_interface/VelocityJointInterface</hardwareInterface>
+        <mechanicalReduction>1</mechanicalReduction>
+      </actuator>
+    </transmission>
   </macro>
 </robot>
