Commit message: Version fonctionnelle avec les rotations des joints chassis/body. Cette version utilise de JointEffortControllers pour les rotations

File: dummiebot_description/urdf/dummiebot.xacro (robot description, xacro)
@@ -129,4 +129,34 @@
     </inertial>
   </link>
+  <transmission name="chassis_body_joint_trans">
+    <type>transmission_interface/SimpleTransmission</type>
+    <joint name="chassis_body_joint">
+      <hardwareInterface>hardware_interface/EffortJointInterface</hardwareInterface>
+    </joint>
+    <actuator name="z_motor">
+      <hardwareInterface>hardware_interface/EffortJointInterface</hardwareInterface>
+      <mechanicalReduction>10</mechanicalReduction>
+    </actuator>
+  </transmission>
+  <transmission name="body_joint_body_trans">
+    <type>transmission_interface/SimpleTransmission</type>
+    <joint name="body_joint_body">
+      <hardwareInterface>hardware_interface/EffortJointInterface</hardwareInterface>
+    </joint>
+    <actuator name="y_motor">
+      <hardwareInterface>hardware_interface/EffortJointInterface</hardwareInterface>
+      <mechanicalReduction>10</mechanicalReduction>
+    </actuator>
+  </transmission>
+  <!--<transmission name="chassis_body_joint_trans">
+    <type>transmission_interface/SimpleTransmission</type>
+    <joint name="chassis_body_joint">
+      <hardwareInterface>EffortJointInterface</hardwareInterface>
+    </joint>
+    <actuator name="z_motor">
+      <hardwareInterface>EffortJointInterface</hardwareInterface>
+      <mechanicalReduction>10</mechanicalReduction>
+    </actuator>
+  </transmission>-->
 <!--
   <joint name="chassis_virtual1" type="fixed">

Commit message: Ajout de la caméra

File: dummiebot_description/urdf/dummiebot.xacro (robot description, xacro)
@@ -19,4 +19,6 @@
   <xacro:property name="body_joint_radius" value="0.1"/>
   <xacro:property name="body_joint_mass" value="1"/>
+  <xacro:property name="camera_size" value="0.05"/>
+  <xacro:property name="camera_mass" value="1"/>
   <!-- Inclusions -->
   <xacro:include filename="$(find dummiebot_description)/urdf/dummiebot.gazebo"/>
@@ -127,4 +129,29 @@
       <mass value="${body_mass}"/>
       <box_inertia m="${body_mass}" x="${body_length}" y="${body_width}" z="${body_height}"/>
+    </inertial>
+  </link>
+  <joint name="body_camera" type="fixed">
+    <parent link="body"/>
+    <child link="camera_link"/>
+    <origin xyz="${-body_length / 2} 0 ${body_height / 2}" rpy="0 0 ${PI}"/>
+  </joint>
+  <link name="camera_link">
+    <collision>
+      <origin xyz="0 0 0" rpy="0 0 0"/>
+      <geometry>
+        <box size="${camera_size} ${camera_size} ${camera_size}"/>
+      </geometry>
+    </collision>
+    <visual>
+      <origin xyz="0 0 0" rpy="0 0 0"/>
+      <geometry>
+        <box size="${camera_size} ${camera_size} ${camera_size}"/>
+      </geometry>
+      <material name="blue"/>
+    </visual>
+    <inertial>
+      <mass value="${camera_mass}"/>
+      <origin xyz="0 0 0" rpy="0 0 0"/>
+      <box_inertia m="${camera_mass}" x="${camera_size}" y="${camera_size}" z="${camera_size}"/>
     </inertial>
   </link>

File: dummiebot_description/urdf/macros.xacro (robot description, xacro)
@@ -49,4 +49,5 @@
     <joint name="${lr}_wheel_hinge" type="continuous">
       <!--<type>transmission_interface/SimpleTransmission</type>-->
+      <type>transmission_interface/SimpleTransmission</type>
       <parent link="chassis"/>
       <child link="${lr}_wheel"/>

Commit message: Déplacement de la caméra à l'avant du robot

File: dummiebot_description/urdf/dummiebot.xacro (robot description, xacro)
@@ -134,5 +134,5 @@
     <parent link="body"/>
     <child link="camera_link"/>
-    <origin xyz="${-body_length / 2} 0 ${body_height / 2}" rpy="0 0 ${PI}"/>
+    <origin xyz="${body_length / 2} 0 ${body_height / 2}" rpy="0 0 0"/>
   </joint>
   <link name="camera_link">

Commit message: Version fonctionnelle avec camera et laser fonctionnels sur Rviz

File: dummiebot_description/urdf/dummiebot.xacro (robot description, xacro)
@@ -156,4 +156,29 @@
     </inertial>
   </link>
+  <joint name="hokuyo_joint" type="fixed">
+    <origin xyz="${chassis_length / 2} 0 ${chassis_height}" rpy="0 0 0"/>
+    <parent link="chassis"/>
+    <child link="hokuyo_link"/>
+  </joint>
+  <!-- Hokuyo Laser -->
+  <link name="hokuyo_link">
+    <collision>
+      <origin xyz="0 0 0" rpy="0 0 0"/>
+      <geometry>
+	       <box size="0.1 0.1 0.1"/>
+      </geometry>
+    </collision>
+    <visual>
+      <origin xyz="0 0 0" rpy="0 0 0"/>
+      <geometry>
+        <mesh filename="package://rrbot_description/meshes/hokuyo.dae"/>
+      </geometry>
+    </visual>
+    <inertial>
+      <mass value="1e-5" />
+      <origin xyz="0 0 0" rpy="0 0 0"/>
+      <inertia ixx="1e-6" ixy="0" ixz="0" iyy="1e-6" iyz="0" izz="1e-6" />
+    </inertial>
+  </link>
   <transmission name="chassis_body_joint_trans">
     <type>transmission_interface/SimpleTransmission</type>

Commit message: Ajout de commentaires et suppressions de fichiers non utilisés

File: dummiebot_description/urdf/dummiebot.xacro (robot description, xacro)
@@ -6,5 +6,5 @@
   <xacro:property name="chassis_length" value="0.6"/>
   <xacro:property name="chassis_width" value="0.5"/>
-  <xacro:property name="chassis_mass" value="50"/>
+  <xacro:property name="chassis_mass" value="5"/>
   <xacro:property name="caster_radius" value="0.05"/>
   <xacro:property name="caster_mass" value="5"/>
@@ -201,65 +201,3 @@
     </actuator>
   </transmission>
-  <!--<transmission name="chassis_body_joint_trans">
-    <type>transmission_interface/SimpleTransmission</type>
-    <joint name="chassis_body_joint">
-      <hardwareInterface>EffortJointInterface</hardwareInterface>
-    </joint>
-    <actuator name="z_motor">
-      <hardwareInterface>EffortJointInterface</hardwareInterface>
-      <mechanicalReduction>10</mechanicalReduction>
-    </actuator>
-  </transmission>-->
-<!--
-  <joint name="chassis_virtual1" type="fixed">
-    <parent link="chassis"/>
-    <child link="virtual1"/>
-    <origin xyz="0 0 ${chassis_height + caster_radius * 2}" rpy="0 0 0"/>
-  </joint>
-  <link name="virtual1">
-    <inertial>
-      <mass value="0.01"/>
-      <sphere_inertia m="0.01" r="0.1"/>
-    </inertial>
-  </link>
-  <joint name="virtual1_virtual2" type="revolute">
-    <parent link="virtual1"/>
-    <child link="virtual2"/>
-    <axis xyz="0 0 1"/>
-    <limit effort="1000.0" lower="-${PI/2}" upper="${PI/2}" velocity="0.5"/>
-  </joint>
-  <link name="virtual2">
-    <inertial>
-      <mass value="0.01"/>
-      <sphere_inertia m="0.01" r="0.1"/>
-    </inertial>
-  </link>
-  <joint name="virtual2_body" type="revolute">
-    <parent link="virtual2"/>
-    <child link="body"/>
-    <axis xyz="0 1 0"/>
-    <limit effort="1000.0" lower="-${PI/4}" upper="${PI/4}" velocity="0.5"/>
-    <origin xyz="0 0 0" rpy="0 0 0"/>
-  </joint>
-  <link name="body">
-    <collision>
-      <origin xyz="0 0 ${body_height / 2}" rpy="0 0 0"/>
-      <geometry>
-        <box size="${body_length} ${body_width} ${body_height}"/>
-      </geometry>
-    </collision>
-    <visual>
-      <origin xyz="0 0 ${body_height / 2}" rpy="0 0 0"/>
-      <geometry>
-        <box size="${body_length} ${body_width} ${body_height}"/>
-      </geometry>
-      <material name="white"/>
-    </visual>
-    <inertial>
-      <origin xyz="0 0 ${body_height / 2}" rpy="0 0 0"/>
-      <mass value="${body_mass}"/>
-      <box_inertia m="${body_mass}" x="${body_length}" y="${body_width}" z="${body_height}"/>
-    </inertial>
-  </link>
--->
 </robot>

File: dummiebot_description/urdf/macros.xacro (robot description, xacro)
@@ -1,3 +1,4 @@
 <robot name="dummiebot">
+  <!-- Macros for inertia of different shapes -->
   <macro name="cylinder_inertia" params="m r h">
     <inertia  ixx="${m*(3*r*r+h*h)/12}" ixy="0" ixz="0"
@@ -18,4 +19,5 @@
     />
   </macro>
+  <!-- Macro for the wheels -->
   <macro name="wheel" params="lr tY">
     <link name="${lr}_wheel">
@@ -48,5 +50,4 @@
     </gazebo>
     <joint name="${lr}_wheel_hinge" type="continuous">
-      <!--<type>transmission_interface/SimpleTransmission</type>-->
       <type>transmission_interface/SimpleTransmission</type>
       <parent link="chassis"/>
@@ -55,18 +56,6 @@
       <axis xyz="0 1 0" rpy="0 0 0"/>
       <limit effort="100" velocity="100"/>
-      <joint_properties damping="0.0" friciton="0.0"/>
+      <joint_properties damping="0.0" friciton="0.5"/>
     </joint>
-<!--
-    <transmission name="${lr}_trans">
-      <type>transmission_interface/SimpleTransmission</type>
-      <joint name="${lr}_wheel_hinge">
-        <hardwareInterface>hardware_interface/EffortJointInterface</hardwareInterface>
-      </joint>
-      <actuator name="${lr}_motor">
-        <hardwareInterface>hardware_interface/EffortJointInterface</hardwareInterface>
-        <mechanicalReduction>1</mechanicalReduction>
-      </actuator>
-    </transmission>
--->
     <transmission name="${lr}_trans">
       <type>transmission_interface/SimpleTransmission</type>

Commit message: Suppression de la variable "ARROW_KEY" dans le programme de contrôle du robot et ajout de contrepoids sur le châssis et le corps du robot

File: dummiebot_description/urdf/dummiebot.xacro (robot description, xacro)
@@ -16,9 +16,9 @@
   <xacro:property name="body_length" value="0.3"/>
   <xacro:property name="body_width" value="0.3"/>
-  <xacro:property name="body_mass" value="0.1"/>
+  <xacro:property name="body_mass" value="1"/>
   <xacro:property name="body_joint_radius" value="0.1"/>
   <xacro:property name="body_joint_mass" value="1"/>
   <xacro:property name="camera_size" value="0.05"/>
-  <xacro:property name="camera_mass" value="1"/>
+  <xacro:property name="camera_mass" value="0.1"/>
   <!-- Inclusions -->
   <xacro:include filename="$(find dummiebot_description)/urdf/dummiebot.gazebo"/>
@@ -51,4 +51,15 @@
     </inertial>
   </link>
+  <joint name="chassis_chassis_counterweight" type="fixed">
+    <parent link="chassis"/>
+    <child link="chassis_counterweight"/>
+    <origin xyz="${-chassis_length / 2} 0 ${chassis_height}" rpy="0 0 0"/>
+  </joint>
+  <link name="chassis_counterweight">
+    <inertial>
+      <mass value="3"/>
+      <box_inertia m="3" x="0" y="0" z="0"/>
+    </inertial>
+  </link>
   <joint name="chassis_caster" type="fixed">
     <parent link="chassis"/>
@@ -156,4 +167,15 @@
     </inertial>
   </link>
+  <joint name="body_body_counterweight" type="fixed">
+    <parent link="body"/>
+    <child link="body_counterweight"/>
+    <origin xyz="${-body_length / 2} 0 ${body_height / 2}" rpy="0 0 0"/>
+  </joint>
+  <link name="body_counterweight">
+    <inertial>
+      <mass value="${camera_mass}"/>
+      <box_inertia m="${camera_mass}" x="0" y="0" z="0"/>
+    </inertial>
+  </link>
   <joint name="hokuyo_joint" type="fixed">
     <origin xyz="${chassis_length / 2} 0 ${chassis_height}" rpy="0 0 0"/>

Commit message: Création d'une map et localisation fonctionnelles

File: dummiebot_description/urdf/dummiebot.xacro (robot description, xacro)
@@ -23,10 +23,9 @@
   <!-- Inclusions -->
   <xacro:include filename="$(find dummiebot_description)/urdf/dummiebot.gazebo"/>
-  <xacro:include filename="$(find dummiebot_description)/urdf/materials.xacro"/>
   <xacro:include filename="$(find dummiebot_description)/urdf/macros.xacro"/>
   <!-- Structure -->
-  <link name="footprint"/>
+  <link name="base_link"/>
   <joint name="base_joint" type="fixed">
-    <parent link="footprint"/>
+    <parent link="base_link"/>
     <child link="chassis"/>
   </joint>
@@ -86,6 +85,6 @@
     </inertial>
   </link>
-  <wheel lr="left" tY="1"/>
-  <wheel lr="right" tY="-1"/>
+  <xacro:wheel lr="left" tY="1"/>
+  <xacro:wheel lr="right" tY="-1"/>
   <joint name="chassis_body_joint" type="revolute">
     <parent link="chassis"/>
@@ -194,5 +193,5 @@
       <origin xyz="0 0 0" rpy="0 0 0"/>
       <geometry>
-        <mesh filename="package://rrbot_description/meshes/hokuyo.dae"/>
+	       <box size="0.1 0.1 0.1"/>
       </geometry>
     </visual>

File: dummiebot_description/urdf/macros.xacro (robot description, xacro)
@@ -1,24 +1,24 @@
-<robot name="dummiebot">
+<robot name="dummiebot" xmlns:xacro="http://ros.org/wiki/xacro">
   <!-- Macros for inertia of different shapes -->
-  <macro name="cylinder_inertia" params="m r h">
+  <xacro:macro name="cylinder_inertia" params="m r h">
     <inertia  ixx="${m*(3*r*r+h*h)/12}" ixy="0" ixz="0"
               iyy="${m*(3*r*r+h*h)/12}" iyz="0"
               izz="${m*r*r/2}"
     />
-  </macro>
-  <macro name="box_inertia" params="m x y z">
+  </xacro:macro>
+  <xacro:macro name="box_inertia" params="m x y z">
     <inertia  ixx="${m*(y*y+z*z)/12}" ixy="0" ixz="0"
               iyy="${m*(x*x+z*z)/12}" iyz="0"
               izz="${m*(x*x+z*z)/12}"
     />
-  </macro>
-  <macro name="sphere_inertia" params="m r">
+  </xacro:macro>
+  <xacro:macro name="sphere_inertia" params="m r">
     <inertia  ixx="${2*m*r*r/5}" ixy="0" ixz="0"
               iyy="${2*m*r*r/5}" iyz="0"
               izz="${2*m*r*r/5}"
     />
-  </macro>
+  </xacro:macro>
   <!-- Macro for the wheels -->
-  <macro name="wheel" params="lr tY">
+  <xacro:macro name="wheel" params="lr tY">
     <link name="${lr}_wheel">
       <collision>
@@ -68,4 +68,4 @@
       </actuator>
     </transmission>
-  </macro>
+  </xacro:macro>
 </robot>

Commit message: Mapping, localisation et navigation fonctionnels

File: dummiebot_description/urdf/dummiebot.xacro (robot description, xacro)
@@ -8,9 +8,9 @@
   <xacro:property name="chassis_mass" value="5"/>
   <xacro:property name="caster_radius" value="0.05"/>
-  <xacro:property name="caster_mass" value="5"/>
-  <xacro:property name="wheel_width" value="0.05"/>
+  <xacro:property name="caster_mass" value="0.1"/>
+  <xacro:property name="wheel_width" value="0.1"/>
   <xacro:property name="wheel_radius" value="0.2"/>
   <xacro:property name="wheel_pos" value="0.2"/>
-  <xacro:property name="wheel_mass" value="5"/>
+  <xacro:property name="wheel_mass" value="0.5"/>
   <xacro:property name="body_height" value="0.6"/>
   <xacro:property name="body_length" value="0.3"/>
@@ -177,11 +177,11 @@
     </inertial>
   </link>
-  <joint name="hokuyo_joint" type="fixed">
+  <!-- Hokuyo Laser 1 -->
+  <joint name="hokuyo1_joint" type="fixed">
     <origin xyz="${chassis_length / 2} 0 ${chassis_height}" rpy="0 0 0"/>
     <parent link="chassis"/>
-    <child link="hokuyo_link"/>
-  </joint>
-  <!-- Hokuyo Laser -->
-  <link name="hokuyo_link">
+    <child link="hokuyo1_link"/>
+  </joint>
+  <link name="hokuyo1_link">
     <collision>
       <origin xyz="0 0 0" rpy="0 0 0"/>
@@ -190,4 +190,29 @@
       </geometry>
     </collision>
+    <visual>
+      <origin xyz="0 0 0" rpy="0 0 0"/>
+      <geometry>
+	       <box size="0.1 0.1 0.1"/>
+      </geometry>
+    </visual>
+    <inertial>
+      <mass value="1e-5" />
+      <origin xyz="0 0 0" rpy="0 0 0"/>
+      <inertia ixx="1e-6" ixy="0" ixz="0" iyy="1e-6" iyz="0" izz="1e-6" />
+    </inertial>
+  </link>
+    <!-- Hokuyo Laser 2 -->
+    <joint name="hokuyo2_joint" type="fixed">
+      <origin xyz="${-chassis_length / 2} 0 ${chassis_height}" rpy="0 0 ${PI}"/>
+      <parent link="chassis"/>
+      <child link="hokuyo2_link"/>
+    </joint>
+    <link name="hokuyo2_link">
+      <collision>
+        <origin xyz="0 0 0" rpy="0 0 0"/>
+        <geometry>
+  	       <box size="0.1 0.1 0.1"/>
+        </geometry>
+      </collision>
     <visual>
       <origin xyz="0 0 0" rpy="0 0 0"/>

File: dummiebot_description/urdf/macros.xacro (robot description, xacro)
@@ -42,9 +42,9 @@
     </link>
     <gazebo reference="${lr}_wheel">
-      <mu1 value="1.0"/>
-      <mu2 value="1.0"/>
-      <kp value="10000000.0"/>
-      <kd value="1.0"/>
-      <fdir1 value="1 0 0"/>
+      <mu1 value="100.0"/>
+      <mu2 value="50.0"/>
+      <!-- <kp value="10000000.0"/>
+      <kd value="100.0"/>
+      <fdir1 value="1 0 0"/> -->
       <material>Gazebo/Black</material>
     </gazebo>
@@ -53,8 +53,8 @@
       <parent link="chassis"/>
       <child link="${lr}_wheel"/>
-      <origin xyz="${-wheel_pos + chassis_length / 2} ${tY * wheel_width / 2 + tY * chassis_width / 2} ${wheel_radius}" rpy="0 0 0"/>
+      <origin xyz="${-wheel_pos + chassis_length / 2} ${tY * wheel_width / 2 + tY * chassis_width / 2 + tY * 0.01} ${wheel_radius}" rpy="0 0 0"/>
       <axis xyz="0 1 0" rpy="0 0 0"/>
       <limit effort="100" velocity="100"/>
-      <joint_properties damping="0.0" friciton="0.5"/>
+      <joint_properties damping="1.0" friciton="0.5"/>
     </joint>
     <transmission name="${lr}_trans">
